Commit message: Agregados controladores de junta y launch de Gazebo

File: urdf/px_trans.urdf (robot description, URDF)
Before this commit: robot px_robot, 7 links, 6 joints
Links:
- link base_link: mass None -> 0.2
- link link1: mass None -> 0.01
- link link2: mass None -> 0.01
- link link3: mass None -> 0.01
- link link4: mass None -> 0.01
